File: Delta DPS-250CP.kicad_sch (KiCad schematic)
At the start: 42 parts, among them IC2 UC3843_DIP8, IC3 LM393, IC501 CQY80NG, Q10 PNP, U1 TOP200YAI

Commit message: Progress
Parts:
- added C1: 470uF, Capacitor_THT:CP_Radial_D8.0mm_P5.00mm, symbol Device:C_Polarized
- added C10: 4700pF, Capacitor_THT:C_Disc_D7.5mm_W5.0mm_P7.50mm, symbol Device:C_Small
- added C11: 220pF, Capacitor_THT:C_Disc_D5.0mm_W2.5mm_P5.00mm, symbol Device:C_Small
- added C2, C6: 47uF, Capacitor_THT:CP_Radial_D8.0mm_P5.00mm, symbol Device:C_Polarized
- added C26, C27: 1nF, Capacitor_THT:C_Disc_D5.0mm_W2.5mm_P5.00mm, symbol Device:C_Small
- added C3: 1nF, Capacitor_THT:C_Disc_D12.5mm_W5.0mm_P10.00mm, symbol Device:C_Small
- added C30: 8200pF, Capacitor_THT:C_Disc_D5.0mm_W2.5mm_P5.00mm, symbol Device:C_Small
- added C4: 100nF, Capacitor_THT:C_Disc_D5.0mm_W2.5mm_P5.00mm, symbol Device:C_Small
- added C5: 1uF, Capacitor_THT:CP_Radial_D8.0mm_P5.00mm, symbol Device:C_Polarized
- added D1, D2: 1N4001, Diode_THT:D_DO-41_SOD81_P5.08mm_Vertical_KathodeUp, symbol Diode:1N4001
- added D17: 1N914, Diode_THT:D_DO-35_SOD27_P7.62mm_Horizontal, symbol Diode:1N914
- added D3, D9: Avalanch, Diode_THT:D_DO-35_SOD27_P7.62mm_Horizontal, symbol Diode:1N914
- added J1: Conn_01x16_Pin, MysteryModule:MysteryModule, symbol Connector:Conn_01x16_Pin
- added L1: L, Inductor_THT:L_Radial_D7.8mm_P5.00mm_Fastron_07HCP, symbol Device:L
- added Q1: 2SK962, Package_TO_SOT_THT:TO-3P-3_Vertical, symbol Component:2SK962
- added R1: 20R, Resistor_THT:R_Radial_Power_L16.1mm_W9.0mm_P7.37mm, symbol Device:R_Small
- added R12, R40: 1k, Resistor_THT:R_Axial_DIN0204_L3.6mm_D1.6mm_P7.62mm_Horizontal, symbol Device:R_Small
- added R13: 0R16, Resistor_THT:R_Axial_DIN0516_L15.5mm_D5.0mm_P5.08mm_Vertical, symbol Device:R_Small
- added R49: 20R, Resistor_THT:R_Axial_DIN0204_L3.6mm_D1.6mm_P7.62mm_Horizontal, symbol Device:R_Small
- added T1: MP-130B, Transformers:MP-130B, symbol Component:MP-130B
- added U2: L78L15_TO92, Package_TO_SOT_THT:TO-92_Inline_Wide, symbol Regulator_Linear:L78L15_TO92
- added U3: L7805, Package_TO_SOT_THT:TO-220-3_Vertical, symbol Regulator_Linear:L7805
- added ZD2: D_Zener, Diode_THT:D_DO-41_SOD81_P7.62mm_Horizontal, symbol Device:D_Zener
- added ZD6: D_Zener, Diode_THT:D_DO-41_SOD81_P5.08mm_Vertical_KathodeUp, symbol Device:D_Zener
- added ZD7: D_Zener, Diode_THT:D_DO-41_SOD81_P10.16mm_Horizontal, symbol Device:D_Zener
- renumbered TR1 to T2, D1 to ZD3
Connections:
- net GNDPWR: now also C27.2, C3.2, C30.2, R13.2, ZD2.2 (A)
- net at D18.2 (A), IC2.4 (RC), R38.2: now also C26.1, C30.1
- net at IC2.3 (CS): now also C26.2, C27.1, R40.2
- net at D15.1 (K), IC2.6 (OUT): now also D17.1 (K), R49.2
- net at IC501.5, R20.1, R29.2: now also ZD2.1 (K)
- net at T2.10: now also D1.2 (A)
- net at T2.6: now also C1.1, D3.1 (K), U3.1 (IN)
- net at T2.7: now also D3.2 (A)
- net at T2.8: now also D2.2 (A)
- net GND: now reaches T2.9
- net GND: now also C1.2, C2.2, C4.2, C5.2, C6.2, U2.2 (GND), U3.2 (GND)
- net at R47.1, R58.1: now also C10.1, C3.1, R1.1, T1.1, ZD6.2 (A)
- new net: C10.2, C11.1, D9.1 (K), R1.2, ZD7.1 (K)
- new net: C11.2, D9.2 (A), Q1.2 (D), T1.4
- new net: Q1.3 (S), R12.2, R13.1, R40.1
- new net: C6.1, L1.2
- new net: D17.2 (A), Q1.1 (G), R12.1, R49.1
- new net: ZD6.1 (K), ZD7.2 (A)
- new net: C5.1, D2.1 (K)
- new net: C4.1, U2.1 (VO)
- new net: C2.1, D1.1 (K), U2.3 (VI)
- new net: L1.1, U3.3 (OUT)
Other:
- moved on the sheet: C31
